File: KiCadProject_Cooker/KiCadProject_Cooker.kicad_pcb (KiCad board)
At the start: 2 copper layers, 10 parts, among them U1 ESP32-WROOM

Commit message: working and functional
Parts:
- moved R1 1.27 mm to (144.8, 61.0)
- turned C1 to 270 degrees
Connections:
- C2 pad 2: Net-(C2-Pad2) -> Net-(C1-Pad2)
- C3 pad 2: Net-(C3-Pad2) -> Net-(C1-Pad2)
- R1 pad 2: Net-(R1-Pad2) -> Net-(C1-Pad2)
- R2 pad 2: Net-(R1-Pad2) -> Net-(C1-Pad2)
- R3 pad 2: Net-(R1-Pad2) -> Net-(C1-Pad2)
- U1 pad 1: Net-(R1-Pad2) -> Net-(C1-Pad2)
- U1 pad 10: Net-(U1-Pad10) -> (no net)
- U1 pad 11: Net-(U1-Pad11) -> (no net)
- U1 pad 12: Net-(U1-Pad12) -> (no net)
- U1 pad 13: Net-(U1-Pad13) -> (no net)
- U1 pad 14: Net-(U1-Pad14) -> (no net)
- U1 pad 15: Net-(U1-Pad15) -> (no net)
- U1 pad 16: Net-(U1-Pad16) -> (no net)
- U1 pad 17: Net-(U1-Pad17) -> (no net)
- U1 pad 18: Net-(U1-Pad18) -> (no net)
- U1 pad 19: Net-(U1-Pad19) -> (no net)
- U1 pad 20: Net-(U1-Pad20) -> (no net)
- U1 pad 21: Net-(U1-Pad21) -> (no net)
- U1 pad 22: Net-(U1-Pad22) -> (no net)
- U1 pad 23: Net-(U1-Pad23) -> (no net)
- U1 pad 24: Net-(U1-Pad24) -> (no net)
- U1 pad 25: Net-(U1-Pad25) -> (no net)
- U1 pad 26: Net-(U1-Pad26) -> (no net)
- U1 pad 27: Net-(U1-Pad27) -> (no net)
- U1 pad 28: Net-(U1-Pad28) -> (no net)
- U1 pad 29: Net-(U1-Pad29) -> (no net)
- U1 pad 3: Net-(U1-Pad3) -> (no net)
- U1 pad 30: Net-(U1-Pad30) -> (no net)
- U1 pad 31: Net-(U1-Pad31) -> (no net)
- U1 pad 32: Net-(U1-Pad32) -> (no net)
- U1 pad 33: Net-(U1-Pad33) -> (no net)
- U1 pad 34: Net-(U1-Pad34) -> (no net)
- U1 pad 35: Net-(U1-Pad35) -> (no net)
- U1 pad 36: Net-(U1-Pad36) -> (no net)
- U1 pad 37: Net-(U1-Pad37) -> (no net)
- U1 pad 38: Net-(U1-Pad38) -> (no net)
- U1 pad 39: Net-(U1-Pad39) -> (no net)
- U1 pad 4: Net-(U1-Pad4) -> (no net)
- U1 pad 5: Net-(U1-Pad5) -> (no net)
- U1 pad 6: Net-(C1-Pad2) -> Net-(C1-Pad1)
- U1 pad 7: Net-(C2-Pad2) -> Net-(C2-Pad1)
- U1 pad 8: Net-(C3-Pad2) -> Net-(C3-Pad1)
- U1 pad 9: Net-(U1-Pad9) -> (no net)
